File: eagle/GBZP.sch (EAGLE design)
At the start: 0 parts

Commit message: Fri 29 Sep 2017 10:20:31 EDT
Parts:
- added BTN_A, BTN_B, BTN_DOWN, BTN_L1, BTN_L2, BTN_LEFT, BTN_R1, BTN_R2, BTN_RIGHT, BTN_SELECT, BTN_START, BTN_UP, BTN_X, BTN_Y: MOMENTARY-SWITCH-SPST-PTH-6.0MM, SparkFun-Switches:MOMENTARY-SWITCH-SPST-PTH-6.0MM
- added CN1: (no value), adafruit:JST_2PIN-SMT
- added LED1: (no value), adafruit:LEDCHIPLED_0805
- added PI1: RPI-ZERO, RPI-Zero:RPI-ZERO
- added POWER1: 03962A, 03962A:03962A
- added R1, R2: 100, adafruit:R-US_R0805
- added S2: (no value), SparkFun-Switches:SWITCH-SPDT-PTH-11.6X4.0MM
- added SCREEN1: GAMEBOYZEROHANDHELDDISPLAYS-2.8, GameboyZeroHandheldDisplays:GAMEBOYZEROHANDHELDDISPLAYS-2.8
Connections:
- new net 3V3: PI1.3V3@1, PI1.3V3@2, R1.2, SCREEN1.VCC
- new net 3V3100OHM: R1.1, SCREEN1.LEDA
- new net A: BTN_A.2, PI1.GPIO19
- new net B: BTN_B.2, PI1.GPIO5
- new net BATT+: CN1.2, POWER1.B+
- new net BATT-: CN1.1, POWER1.B-
- new net CSX: PI1.!CE0!/GPIO8, SCREEN1.CSX
- new net D/CX: PI1.GEN5/GPIO24, SCREEN1.D/CX
- new net DOWN: BTN_DOWN.2, PI1.GPIO12
- new net GND: BTN_A.1, BTN_B.1, BTN_DOWN.1, BTN_L1.1, BTN_L2.1, BTN_LEFT.1, BTN_R1.1, BTN_R2.1, BTN_RIGHT.1, BTN_SELECT.1, BTN_START.1, BTN_UP.1, BTN_X.1, BTN_Y.1, LED1.C, PI1.GND@1, PI1.GND@2, PI1.GND@3, PI1.GND@4, PI1.GND@5, PI1.GND@6, PI1.GND@7, PI1.GND@8, POWER1.OUT-, SCREEN1.GND, SCREEN1.GND2, SCREEN1.LED_K1, SCREEN1.LED_K2, SCREEN1.LED_K3, SCREEN1.LED_K4
- new net L1: BTN_L1.2, PI1.GPIO18
- new net L2: BTN_L2.2, PI1.RXD0/GPIO15
- new net LED: LED1.A, R2.1
- new net LEFT: BTN_LEFT.2, PI1.GPIO21
- new net R1: BTN_R1.2, PI1.GPIO27/GEN2
- new net R2: BTN_R2.2, PI1.GPIO17/GEN0
- new net RESET: PI1.GEN/6GPIO25, SCREEN1.RESET
- new net RIGHT: BTN_RIGHT.2, PI1.GPIO20
- new net SCL: PI1.GPIO11/SCLK, SCREEN1.SCL
- new net SDI: PI1.GPIO10/MOSI, SCREEN1.SDI
- new net SDO: PI1.GPIO9/MISO, SCREEN1.SDO
- new net SELECT: BTN_SELECT.2, PI1.GPIO26
- new net START: BTN_START.2, PI1.GPIO16
- new net SWITCH_IN+: POWER1.OUT+, S2.P
- new net SWITCH_OUT+: PI1.5V0@1, PI1.5V0@2, R2.2, S2.O
- new net UP: BTN_UP.2, PI1.!CE!/GPIO7
- new net X: BTN_X.2, PI1.GPIO6
- new net Y: BTN_Y.2, PI1.GPIO13
Other:
- note added: "BATTERY"
- note added: "D-PAD BUTTONS"
- note added: "DISPLAY"
- note added: "FACE BUTTONS"
- note added: "FUNCTION BUTTONS"
- note added: "LED"
- note added: "POWER"
- note added: "RASPBERRY PI"
- note added: "SHOULDER BUTTONS"
- note added: "SWITCH"
