File: eagle/GBZP.sch (EAGLE design)
At the start: 32 parts, among them J1 AUDIO_JACK_3.5MM_SMD, U1 LM4875

Commit message: Tue 31 Oct 2017 16:24:12 EDT
Parts:
- BTN_SELECT, BTN_START: value MOMENTARY-SWITCH-SPST-SMD-6.0X3.5MM -> MOMENTARY-SWITCH-SPST-SMD-6.2MM-TALL; device SparkFun-Switches:MOMENTARY-SWITCH-SPST-SMD-6.0X3.5MM -> SparkFun-Switches:MOMENTARY-SWITCH-SPST-SMD-6.2MM-TALL
- J1: value AUDIO_JACK_3.5MM_SMD -> AUDIO_JACK_3.5MM_PTH; device SparkFun-Connectors:AUDIO_JACK_3.5MM_SMD -> SparkFun-Connectors:AUDIO_JACK_3.5MM_PTH
Connections:
- net L1: now also PI1.ID_SC; no longer PI1.GPIO21

Commit message: Mon  6 Nov 2017 08:50:14 EST
Parts:
- BTN_A, BTN_B, BTN_DOWN, BTN_L1, BTN_LEFT, BTN_R1, BTN_RIGHT, BTN_SELECT, BTN_START, BTN_UP, BTN_X, BTN_Y: value MOMENTARY-SWITCH-SPST-SMD-6.2MM-TALL -> PAD+SWITCH+HOLE; device SparkFun-Switches:MOMENTARY-SWITCH-SPST-SMD-6.2MM-TALL -> pad+switch+hole:PAD+SWITCH+HOLE
Connections:
- removed net PWM_LEFT: PI1.GPIO13
- net A: now also BTN_A.P$ACTIVE, PI1.GPIO19; no longer BTN_A.2, PI1.GPIO16
- net B: now also BTN_B.P$ACTIVE; no longer BTN_B.2
- net DOWN: now also BTN_DOWN.P$ACTIVE; no longer BTN_DOWN.2
- net GND: now also BTN_A.P$GND, BTN_B.P$GND, BTN_DOWN.P$GND, BTN_L1.P$GND, BTN_LEFT.P$GND, BTN_R1.P$GND, BTN_RIGHT.P$GND, BTN_SELECT.P$GND, BTN_START.P$GND, BTN_UP.P$GND, BTN_X.P$GND, BTN_Y.P$GND; no longer BTN_A.1, BTN_B.1, BTN_DOWN.1, BTN_L1.1, BTN_LEFT.1, BTN_R1.1, BTN_RIGHT.1, BTN_SELECT.1, BTN_START.1, BTN_UP.1, BTN_X.1, BTN_Y.1
- net L1: now also BTN_L1.P$ACTIVE, PI1.GPIO26; no longer BTN_L1.2, PI1.ID_SC
- net LEFT: now also BTN_LEFT.P$ACTIVE; no longer BTN_LEFT.2
- net R1: now also BTN_R1.P$ACTIVE; no longer BTN_R1.2
- net RIGHT: now also BTN_RIGHT.P$ACTIVE; no longer BTN_RIGHT.2
- net SELECT: now also BTN_SELECT.P$ACTIVE, PI1.ID_SC; no longer BTN_SELECT.2, PI1.GPIO5
- net START: now also BTN_START.P$ACTIVE, PI1.GPIO6; no longer BTN_START.2, PI1.GPIO19
- net UP: now also BTN_UP.P$ACTIVE; no longer BTN_UP.2
- net X: now also BTN_X.P$ACTIVE, PI1.GPIO16; no longer BTN_X.2, PI1.GPIO26
- net Y: now also BTN_Y.P$ACTIVE, PI1.GPIO5; no longer BTN_Y.2, PI1.GPIO6

Commit message: Sat 11 Nov 2017 12:28:11 EST
Parts:
- renumbered SCREEN1 to ILI9341-TFT-2.8
Connections:
- new net GPIO12: PI1.GPIO12
- new net GPIO16: PI1.GPIO16
- new net GPIO20: PI1.GPIO20
- new net GPIO21: PI1.GPIO21
- new net GPIO23: PI1.GEN4/GPIO23
- new net GPIO5: PI1.GPIO5
- new net GPIO7: PI1.!CE!/GPIO7
- net A: now also PI1.TXD0/GPIO14; no longer PI1.GPIO19
- net B: now also PI1.GPIO27/GEN2; no longer PI1.GPIO12
- net DOWN: now also PI1.GPIO6; no longer PI1.GPIO22/GEN3
- net L1: now also PI1.GPIO2/SDA1; no longer PI1.GPIO26
- net LEFT: now also PI1.GPIO26; no longer PI1.TXD0/GPIO14
- net R1: now also PI1.GPIO3/SCL1; no longer PI1.GPIO20
- net RIGHT: now also PI1.GPIO13; no longer PI1.!CE!/GPIO7
- net SELECT: now also PI1.GPIO22/GEN3; no longer PI1.ID_SC
- net START: now also PI1.RXD0/GPIO15; no longer PI1.GPIO6
- net UP: now also PI1.GPIO19; no longer PI1.GPIO27/GEN2
- net X: now also PI1.GPIO4/GCKL; no longer PI1.GPIO16
- net Y: now also PI1.GPIO17/GEN0; no longer PI1.GPIO5
