File: eagle/GBZP.brd (EAGLE design)
At the start: 69.5 x 114.2 mm, 29 parts, among them J1 AUDIO_JACK_3.5MM_SMD

Commit message: Sun Oct  1 17:41:23 EDT 2017
Parts:
- moved BTN_START 27.0 mm to (40.7, 15.0)
- moved BTN_SELECT 26.5 mm to (29.1, 15.0)
- moved PI1 8.66 mm to (71.3, 112.4)
- moved BTN_DOWN 2.24 mm to (12.5, 29.1)
- moved BTN_LEFT 2.24 mm to (4.53, 37.0), turned to 90 degrees
- moved BTN_RIGHT 2.24 mm to (20.4, 37.0), turned to 270 degrees
- moved BTN_UP 2.24 mm to (12.5, 45.0)

Commit message: Sun Oct  1 21:02:41 EDT 2017
Parts:
- moved U$1 4.00 mm to (10.0, 112.0)
Other:
- outline, holes or cut-outs redrawn
Changed lines of the file:
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@@
 <layer number="17" name="Pads" color="2" fill="1" visible="yes" active="yes"/>
 <layer number="18" name="Vias" color="2" fill="1" visible="yes" active="yes"/>
-<layer number="19" name="Unrouted" color="6" fill="1" visible="no" active="yes"/>
+<layer number="19" name="Unrouted" color="6" fill="1" visible="yes" active="yes"/>
 <layer number="20" name="Dimension" color="15" fill="1" visible="yes" active="yes"/>
 <layer number="21" name="tPlace" color="7" fill="1" visible="yes" active="yes"/>
@@
 <wire x1="35.45" y1="15.01" x2="37.71" y2="12.75" width="0.0762" layer="51" curve="90"/>
 <wire x1="35.45" y1="15.01" x2="37.81" y2="17.37" width="0.0762" layer="51" curve="-90"/>
+<circle x="2.5" y="24.83" radius="1.2" width="0.0762" layer="20"/>
+<circle x="2.5" y="62.43" radius="1.2" width="0.0762" layer="20"/>
+<circle x="2.5" y="108.1" radius="1.2" width="0.0762" layer="20"/>
+<circle x="67" y="108.1" radius="1.2" width="0.0762" layer="20"/>
+<circle x="67" y="62.43" radius="1.2" width="0.0762" layer="20"/>
+<circle x="67" y="27.5" radius="1.2" width="0.0762" layer="20"/>
+<circle x="56.76" y="32.6" radius="1.2" width="0.0762" layer="20"/>
+<circle x="46.99" y="22.29" radius="1.2" width="0.0762" layer="20"/>
+<circle x="29.83" y="33.29" radius="1.2" width="0.0762" layer="20"/>
+<circle x="24.33" y="27.45" radius="1.2" width="0.0762" layer="20"/>
+<circle x="23.45" y="23.58" radius="1.2" width="0.0762" layer="20"/>
 </plain>
 <attributes>
@@
 <element name="C3" library="adafruit" library_urn="urn:adsk.eagle:library:420" package="C0805" value="33nF" x="33" y="8" rot="MR0"/>
 <element name="C4" library="adafruit" library_urn="urn:adsk.eagle:library:420" package="C0805" value="33nF" x="48" y="11" rot="MR180"/>
-<element name="U$1" library="SparkFun-Retired" library_urn="urn:adsk.eagle:library:533" package="KPS-1290" value="SWITCH_SPDT" x="6" y="112" rot="MR180">
-<attribute name="PROD_ID" value="SWCH-10651" x="6" y="112" size="1.778" layer="28" rot="MR180" display="off"/>
+<element name="U$1" library="SparkFun-Retired" library_urn="urn:adsk.eagle:library:533" package="KPS-1290" value="SWITCH_SPDT" x="10" y="112" rot="MR180">
+<attribute name="PROD_ID" value="SWCH-10651" x="10" y="112" size="1.778" layer="28" rot="MR180" display="off"/>
 </element>
 </elements>
@@
 <contactref element="U$1" pad="O"/>
 <wire x1="43.487" y1="101.448" x2="43.487" y2="103.988" width="0" layer="19" extent="16-16"/>
-<wire x1="3.75" y1="109.75" x2="43.487" y2="103.988" width="0" layer="19" extent="16-16"/>
-<wire x1="7.5" y1="55" x2="3.75" y2="109.75" width="0" layer="19" extent="1-16"/>
+<wire x1="7.75" y1="109.75" x2="43.487" y2="103.988" width="0" layer="19" extent="16-16"/>
+<wire x1="7.5" y1="55" x2="7.75" y2="109.75" width="0" layer="19" extent="1-16"/>
 </signal>
 <signal name="BATT+">
@@
 <contactref element="POWER1" pad="OUT+"/>
 <contactref element="U$1" pad="P"/>
-<wire x1="25.65" y1="87.35" x2="6.75" y2="109.75" width="0" layer="19" extent="16-16"/>
+<wire x1="25.65" y1="87.35" x2="10.75" y2="109.75" width="0" layer="19" extent="16-16"/>
 </signal>
 <signal name="L1">

Commit message: clean up
Parts:
- moved PI1 69.3 mm to (2.00, 113.0), turned to 180 degrees
- moved POWER1 43.3 mm to (42.5, 62.6), turned to 90 degrees
- moved CN1 28.6 mm to (33.6, 76.0), turned to 270 degrees
- moved LED1 0.50 mm to (3.00, 55.0)
- moved R2 0.50 mm to (7.00, 55.0)

Commit message: clean up
Parts:
- moved C2 2.00 mm to (31.0, 12.0)
- moved C3 2.00 mm to (31.0, 8.00)
- moved R4 2.00 mm to (31.0, 6.00)
- moved R5 2.00 mm to (31.0, 10.0)
- moved J1 1.65 mm to (39.1, 1.00)
- moved U$1 1.21 mm to (11.1, 111.5)
- moved BTN_SELECT 1.00 mm to (29.1, 16.0)
- moved BTN_START 1.00 mm to (40.7, 16.0)
- moved C1 1.00 mm to (47.0, 7.00)
- moved C4 1.00 mm to (47.0, 11.0)
- moved R3 1.00 mm to (47.0, 13.0)
- moved R6 1.00 mm to (47.0, 9.00)
- moved BTN_LEFT 0.36 mm to (4.20, 36.9)
- moved BTN_DOWN 0.34 mm to (12.2, 28.9)
- moved BTN_UP 0.30 mm to (12.2, 44.9), turned to 90 degrees
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Other:
- outline, holes or cut-outs redrawn
