File: eagle/gameboy-macro.brd (EAGLE design)
At the start: 160 x 62 mm, 32 parts, among them J1 AUDIO_JACK_3.5MM_PTH, U1 LM4875

Commit message: Tue 21 Nov 2017 18:24:16 EST
Parts:
- R10: value 27k -> EVU-TUHB07C54
- moved R1 13.0 mm to (117.0, 47.0), turned to 270 degrees
- moved C3 7.43 mm to (126.0, 23.5), turned to 180 degrees
- moved C4 4.00 mm to (126.0, 21.0), turned to 180 degrees
- moved R3 2.53 mm to (126.0, 18.5), turned to 180 degrees
- moved R10 1.03 mm to (131.0, 11.5)
- moved C10 1.00 mm to (152.0, 14.0)
- moved C11 1.00 mm to (141.0, 14.0)
- moved C12 1.00 mm to (144.0, 14.0)
- moved C2 1.00 mm to (148.0, 21.0)
- moved J1 1.00 mm to (145.1, 3.50)
- moved J2 1.00 mm to (143.0, 21.0)
- moved LED1 1.00 mm to (39.0, 5.00)
- moved R2 1.00 mm to (43.0, 5.00)
- moved R5 1.00 mm to (147.0, 14.0)
- moved U1 1.00 mm to (137.0, 26.0)
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Connections:
- removed net GPIO23: PCB1.P$16
- new net GPIO15: PCB1.P$10
- net A: now also PCB1.P$7; no longer PCB1.P$8
- net B: now also PCB1.P$8; no longer PCB1.P$13
- net DOWN: now also PCB1.P$37; no longer PCB1.P$31
- net L1: now also PCB1.P$5; no longer PCB1.P$3
- net LEFT: now also PCB1.P$35; no longer PCB1.P$37
- net R1: now also PCB1.P$3; no longer PCB1.P$5
- net START: now also PCB1.P$16; no longer PCB1.P$10
- net UP: now also PCB1.P$31; no longer PCB1.P$35
- net X: now also PCB1.P$11; no longer PCB1.P$7
- net Y: now also PCB1.P$13; no longer PCB1.P$11
Routing:
- net SWITCH_OUT+: track 6.15 -> 226.6 mm, vias 0 -> 3
- net UP: track 0.00 -> 103.7 mm
- net LEFT: track 0.00 -> 98.6 mm
- net SELECT: track 0.00 -> 96.3 mm, vias 0 -> 2
- net 3V3: track 0.00 -> 95.8 mm, vias 0 -> 2
- net RIGHT: track 0.00 -> 85.1 mm
- net START: track 0.00 -> 84.8 mm, vias 0 -> 2
- net X: track 0.00 -> 82.1 mm
- net DOWN: track 0.00 -> 80.0 mm
- net L1: track 0.00 -> 75.0 mm
- net Y: track 0.00 -> 64.6 mm
- net A: track 0.00 -> 59.0 mm
- net SWITCH_IN+: track 0.00 -> 57.8 mm
- net R1: track 0.00 -> 54.9 mm
- net B: track 0.00 -> 44.1 mm
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
Commit message: Tue 21 Nov 2017 18:40:45 EST
Parts:
- added U$4, U$5, U$6, U$7: (no value), holes:2,8
- R2: value 220 -> 1K
- moved BTN_SELECT 2.00 mm to (14.0, 8.00)
- moved BTN_START 2.00 mm to (26.0, 8.00)
- moved S1 2.00 mm to (31.0, 61.0)
Routing:
- net START: track 84.8 -> 82.8 mm
- net SWITCH_OUT+: track 226.6 -> 228.6 mm
- net SWITCH_IN+: track 57.8 -> 59.8 mm
- net SELECT: track 96.3 -> 94.3 mm
Other:
- board size 160 x 62 mm -> 160 x 64 mm
Changed lines of the file:
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@@
 <board>
 <plain>
-<wire x1="0" y1="10" x2="0" y2="59.5" width="0.254" layer="20"/>
-<wire x1="0" y1="59.5" x2="2.5" y2="62" width="0.254" layer="20" curve="-90"/>
-<wire x1="2.5" y1="62" x2="157.5" y2="62" width="0.254" layer="20"/>
-<wire x1="157.5" y1="62" x2="160" y2="59.5" width="0.254" layer="20" curve="-90"/>
-<wire x1="160" y1="59.5" x2="160" y2="10" width="0.254" layer="20"/>
+<wire x1="0" y1="10" x2="0" y2="61.5" width="0.254" layer="20"/>
+<wire x1="0" y1="61.5" x2="2.5" y2="64" width="0.254" layer="20" curve="-90"/>
+<wire x1="2.5" y1="64" x2="157.5" y2="64" width="0.254" layer="20"/>
+<wire x1="157.5" y1="64" x2="160" y2="61.5" width="0.254" layer="20" curve="-90"/>
+<wire x1="160" y1="61.5" x2="160" y2="10" width="0.254" layer="20"/>
 <wire x1="160" y1="10" x2="150" y2="0" width="0.254" layer="20" curve="-90"/>
 <wire x1="150" y1="0" x2="10" y2="0" width="0.254" layer="20"/>
 <wire x1="10" y1="0" x2="0" y2="10" width="0.254" layer="20" curve="-90"/>
+<wire x1="0" y1="10" x2="0" y2="61.5" width="0" layer="51"/>
+<wire x1="0" y1="61.5" x2="2.5" y2="64" width="0" layer="51" curve="-90"/>
+<wire x1="2.5" y1="64" x2="157.5" y2="64" width="0" layer="51"/>
+<wire x1="157.5" y1="64" x2="160" y2="61.5" width="0" layer="51" curve="-90"/>
+<wire x1="160" y1="61.5" x2="160" y2="10" width="0" layer="51"/>
+<wire x1="160" y1="10" x2="150" y2="0" width="0" layer="51" curve="-90"/>
+<wire x1="150" y1="0" x2="10" y2="0" width="0" layer="51"/>
+<wire x1="10" y1="0" x2="0" y2="10" width="0" layer="51" curve="-90"/>
+<wire x1="37.25" y1="61" x2="114.75" y2="61" width="0" layer="51"/>
+<wire x1="114.75" y1="61" x2="114.75" y2="7" width="0" layer="51"/>
+<wire x1="114.75" y1="7" x2="37.25" y2="7" width="0" layer="51"/>
+<wire x1="37.25" y1="7" x2="37.25" y2="61" width="0" layer="51"/>
 </plain>
 <attributes>
@@
 <element name="BTN_Y" library="pad+switch+hole" package="PAD+SWITCH" value="PAD+SWITCH" x="126.42" y="46.21" smashed="yes" rot="R180"/>
 <element name="BTN_A" library="pad+switch+hole" package="PAD+SWITCH" value="PAD+SWITCH" x="137.42" y="37.21" smashed="yes" rot="R180"/>
-<element name="BTN_B" library="pad+switch+hole" package="PAD+SWITCH" value="PAD+SWITCH" x="123.42" y="31.21" smashed="yes" rot="R180"/>
+<element name="BTN_B" library="pad+switch+hole" package="PAD+SWITCH" value="PAD+SWITCH" x="123.42" y="31.21" rot="R180"/>
 <element name="BTN_L1" library="pad+switch+hole" package="PAD+SWITCH" value="PAD+SWITCH" x="151.47" y="41.7" smashed="yes" rot="R180"/>
 <element name="BTN_R1" library="pad+switch+hole" package="PAD+SWITCH" value="PAD+SWITCH" x="148.42" y="27.21" smashed="yes" rot="R180"/>
-<element name="BTN_START" library="pad+switch+hole" package="PAD+SWITCH" value="PAD+SWITCH" x="24" y="8" smashed="yes"/>
-<element name="BTN_SELECT" library="pad+switch+hole" package="PAD+SWITCH" value="PAD+SWITCH" x="12" y="8" smashed="yes"/>
-<element name="R2" library="adafruit" package="R0805" value="220" x="43" y="5"/>
+<element name="BTN_START" library="pad+switch+hole" package="PAD+SWITCH" value="PAD+SWITCH" x="26" y="8" smashed="yes"/>
+<element name="BTN_SELECT" library="pad+switch+hole" package="PAD+SWITCH" value="PAD+SWITCH" x="14" y="8" smashed="yes"/>
+<element name="R2" library="adafruit" package="R0805" value="1K" x="43" y="5"/>
 <element name="LED1" library="adafruit" package="CHIPLED_0805" value="Blue" x="39" y="5" rot="R90"/>
 <element name="BTN_UP" library="pad+switch+hole" package="PAD+SWITCH" value="PAD+SWITCH" x="18" y="51" smashed="yes"/>
@@
 </element>
 <element name="PCB1" library="e14_Rpi3_RevA+mirror-pcb-no-silk" package="RPI3" value="RPI3RPI3" x="122" y="56" rot="R180"/>
-<element name="S1" library="adafruit" package="EG1213" value="EG1213" x="31" y="59" rot="R180"/>
+<element name="S1" library="adafruit" package="EG1213" value="EG1213" x="31" y="61" rot="R180"/>
+<element name="U$4" library="holes" library_urn="urn:adsk.eagle:library:237" package="2,8" package3d_urn="urn:adsk.eagle:package:14271/1" value="" x="4" y="60"/>
+<element name="U$5" library="holes" library_urn="urn:adsk.eagle:library:237" package="2,8" package3d_urn="urn:adsk.eagle:package:14271/1" value="" x="156" y="60"/>
+<element name="U$6" library="holes" library_urn="urn:adsk.eagle:library:237" package="2,8" package3d_urn="urn:adsk.eagle:package:14271/1" value="" x="155" y="7"/>
+<element name="U$7" library="holes" library_urn="urn:adsk.eagle:library:237" package="2,8" package3d_urn="urn:adsk.eagle:package:14271/1" value="" x="5" y="7"/>
 </elements>
 <signals>
@@
 <polygon width="0.254" layer="1">
 <vertex x="0" y="10"/>
-<vertex x="0" y="59.5" curve="-90"/>
-<vertex x="2.5" y="62"/>
-<vertex x="157.5" y="62" curve="-90"/>
-<vertex x="160" y="59.5"/>
+<vertex x="0" y="61.5" curve="-90"/>
+<vertex x="2.5" y="64"/>
+<vertex x="157.5" y="64" curve="-90"/>
+<vertex x="160" y="61.5"/>
 <vertex x="160" y="10" curve="-90"/>
 <vertex x="150" y="0"/>
@@
 <polygon width="0.254" layer="16">
 <vertex x="160" y="10"/>
-<vertex x="160" y="59.5" curve="90"/>
-<vertex x="157.5" y="62"/>
-<vertex x="2.5" y="62" curve="90"/>
-<vertex x="0" y="59.5"/>
+<vertex x="160" y="61.5" curve="90"/>
+<vertex x="157.5" y="64"/>
+<vertex x="2.5" y="64" curve="90"/>
+<vertex x="0" y="61.5"/>
 <vertex x="0" y="10" curve="90"/>
 <vertex x="10" y="0"/>
@@
 <wire x1="79" y1="15" x2="64" y2="15" width="0.254" layer="16"/>
 <via x="64" y="15" extent="1-16" drill="0.5"/>
-<wire x1="64" y1="15" x2="14.475" y2="15" width="0.254" layer="1"/>
-<wire x1="14.475" y1="15" x2="14.475" y2="10.365" width="0.254" layer="1"/>
+<wire x1="64" y1="15" x2="16.475" y2="15" width="0.254" layer="1"/>
+<wire x1="16.475" y1="15" x2="16.475" y2="10.365" width="0.254" layer="1"/>
 <wire x1="95.8634" y1="15" x2="79" y2="15" width="0.254" layer="1"/>
 </signal>
@@
 <wire x1="78" y1="14" x2="65" y2="14" width="0.254" layer="16"/>
 <via x="65" y="14" extent="1-16" drill="0.5"/>
-<wire x1="65" y1="14" x2="26.475" y2="14" width="0.254" layer="1"/>
-<wire x1="26.475" y1="14" x2="26.475" y2="10.365" width="0.254" layer="1"/>
+<wire x1="65" y1="14" x2="28.475" y2="14" width="0.254" layer="1"/>
+<wire x1="28.475" y1="14" x2="28.475" y2="10.365" width="0.254" layer="1"/>
 <wire x1="94.6" y1="14" x2="78" y2="14" width="0.254" layer="1"/>
 </signal>
@@
 <wire x1="135" y1="13.5" x2="135" y2="13.15" width="0.254" layer="16"/>
 <wire x1="135" y1="13.15" x2="141" y2="13.15" width="0.254" layer="16"/>
-<wire x1="33" y1="59" x2="33" y2="38" width="0.254" layer="16"/>
+<wire x1="33" y1="61" x2="33" y2="38" width="0.254" layer="16"/>
 <wire x1="33" y1="38" x2="59" y2="38" width="0.254" layer="16"/>
 <wire x1="113.6434" y1="2.2282" x2="112.35" y2="2.2282" width="0.254" layer="1"/>
@@
 <contactref element="POWER1" pad="OUT+"/>
 <contactref element="S1" pad="2"/>
-<wire x1="31" y1="59" x2="31" y2="36" width="0.254" layer="16"/>
+<wire x1="31" y1="61" x2="31" y2="36" width="0.254" layer="16"/>
 <wire x1="55.65" y1="36" x2="55.65" y2="25.9" width="0.254" layer="16"/>
 <wire x1="31" y1="36" x2="55.65" y2="36" width="0.254" layer="16"/>

Commit message: Wed 22 Nov 2017 16:59:29 EST
Parts:
- BTN_A, BTN_B, BTN_DOWN, BTN_L1, BTN_LEFT, BTN_R1, BTN_RIGHT, BTN_SELECT, BTN_START, BTN_UP, BTN_X, BTN_Y: value PAD+SWITCH -> GAMEBOY-ZERO-BUTTON; device pad+switch+hole:PAD+SWITCH -> GameboyZeroButtonLibrary:GAMEBOY-ZERO-BUTTON
- moved BTN_SELECT 3.61 mm to (12.0, 11.0)
- moved BTN_START 3.61 mm to (24.0, 11.0)
- moved J3 2.00 mm to (33.0, 6.00)
- moved U$6 2.00 mm to (155.0, 5.00)
- moved U$7 2.00 mm to (5.00, 5.00)
- moved U$4 1.41 mm to (5.00, 59.0)
- moved U$5 1.41 mm to (155.0, 59.0)
- moved C10 1.00 mm to (152.0, 15.0)
- moved C11 1.00 mm to (141.0, 15.0)
- moved C12 1.00 mm to (144.0, 15.0)
- moved J1 1.00 mm to (145.1, 4.50), flipped to the bottom
- moved R5 1.00 mm to (147.0, 15.0)
Routing:
- net CAP_LINE_JACK: track 29.5 -> 26.4 mm
- net BATT-: track 25.2 -> 27.2 mm
- net BATT+: track 34.2 -> 36.2 mm
- net SELECT: track 94.3 -> 93.3 mm
- net HEADPHONES: track 48.8 -> 47.8 mm
- net CAP_LINE: track 18.8 -> 17.8 mm
- net BYP: track 26.1 -> 25.1 mm
- net START: track 82.8 -> 81.8 mm
Other:
- outline, holes or cut-outs redrawn
