File: eagle/gameboy-macro.brd (EAGLE design)
At the start: 160 x 64 mm, 36 parts, among them J1 AUDIO_JACK_3.5MM_PTH, U1 LM4875

Commit message: Tue 28 Nov 2017 19:11:42 EST - ITS MACRO TIME
Routing:
- net VOUT1: track 17.5 -> 16.6 mm
Changed lines of the file:
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@@
 <layer number="220" name="220bmp" color="21" fill="1" visible="no" active="no"/>
 <layer number="221" name="221bmp" color="22" fill="1" visible="no" active="no"/>
+<layer number="222" name="222bmp" color="23" fill="1" visible="no" active="no"/>
 <layer number="223" name="223bmp" color="24" fill="1" visible="no" active="no"/>
 <layer number="224" name="224bmp" color="25" fill="1" visible="no" active="no"/>
@@
 <wire x1="114.75" y1="7" x2="37.25" y2="7" width="0" layer="51"/>
 <wire x1="37.25" y1="7" x2="37.25" y2="61" width="0" layer="51"/>
-<polygon width="0.1524" layer="51">
-<vertex x="170" y="0"/>
-<vertex x="170" y="51"/>
-<vertex x="235" y="51"/>
-<vertex x="235" y="0"/>
-</polygon>
 </plain>
 <attributes>
@@
 <contactref element="U1" pad="5"/>
 <contactref element="J2" pad="1"/>
-<wire x1="139.6" y1="27.905" x2="146.6" y2="27.905" width="0.254" layer="16"/>
-<wire x1="146.6" y1="21" x2="146.6" y2="27.905" width="0.254" layer="16"/>
-<wire x1="143" y1="21" x2="146.6" y2="21" width="0.254" layer="16"/>
+<wire x1="146.6" y1="21" x2="143" y2="21" width="0.254" layer="16"/>
+<wire x1="146.6" y1="26.3528875" x2="146.6" y2="21" width="0.254" layer="16"/>
+<wire x1="139.6" y1="27.905" x2="145.0478875" y2="27.905" width="0.254" layer="16"/>
+<wire x1="145.0478875" y1="27.905" x2="146.6" y2="26.3528875" width="0.254" layer="16"/>
 </signal>
 <signal name="N$2">
