File: eagle/gameboy-macro.sch (EAGLE design)
At the start: 32 parts, among them J1 AUDIO_JACK_3.5MM_PTH, U1 LM4875

Commit message: Tue 21 Nov 2017 18:40:45 EST
Parts:
- R2: value 220 -> 1K
Changed lines of the file:
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@@
 <part name="BTN_L1" library="pad+switch+hole" deviceset="PAD+SWITCH" device="" value="PAD+SWITCH"/>
 <part name="BTN_R1" library="pad+switch+hole" deviceset="PAD+SWITCH" device="" value="PAD+SWITCH"/>
-<part name="R2" library="adafruit" deviceset="R-US_" device="R0805" value="220"/>
+<part name="R2" library="adafruit" deviceset="R-US_" device="R0805" value="1K"/>
 <part name="LED1" library="adafruit" deviceset="LED" device="CHIPLED_0805" value="Blue"/>
 <part name="GND12" library="supply1" library_urn="urn:adsk.eagle:library:371" deviceset="GND" device=""/>
@@
 <pinref part="J2" gate="G$1" pin="1"/>
 <wire x1="294.64" y1="27.94" x2="292.1" y2="27.94" width="0.1524" layer="91"/>
-<label x="292.1" y="27.94" size="1.27" layer="95" rot="MR0"/>
+<label x="292.1" y="27.94" size="1.016" layer="95" rot="MR0"/>
 </segment>
 </net>
@@
 <pinref part="J2" gate="G$1" pin="2"/>
 <wire x1="294.64" y1="25.4" x2="292.1" y2="25.4" width="0.1524" layer="91"/>
-<label x="292.1" y="25.4" size="1.27" layer="95" rot="MR0"/>
-</segment>
-</net>
+<label x="292.1" y="25.4" size="1.016" layer="95" rot="MR0"/>
+</segment>
+</net>

Commit message: Wed 22 Nov 2017 16:59:29 EST
Parts:
- BTN_A, BTN_B, BTN_DOWN, BTN_L1, BTN_LEFT, BTN_R1, BTN_RIGHT, BTN_SELECT, BTN_START, BTN_UP, BTN_X, BTN_Y: value PAD+SWITCH -> GAMEBOY-ZERO-BUTTON; device pad+switch+hole:PAD+SWITCH -> GameboyZeroButtonLibrary:GAMEBOY-ZERO-BUTTON
