File: eagle/gameboy-pocket.brd (EAGLE design)
At the start: 71.2 x 116.5 mm, 32 parts, among them U1 LM4875, X1 STEREOJACK

Commit message: =Fri Mar  9 07:52:40 EST 2018
Parts:
- removed R5: 1KOhm, adafruit:R0805
- R3: value 1KOhm -> 100K
- moved R4 29.4 mm to (48.2, 11.0), turned to 270 degrees
- moved C1 3.00 mm to (20.5, 8.40)
Connections:
- removed net HPHONE: R5.1, U1.3
- net DC_VOL: now also R10.3; no longer R10.5
- net HEADPHONES: now also U1.3; no longer R5.2, X1.4
- net SWITCH_OUT+: now also R10.5; no longer R10.3
Routing:
- net SWITCH_OUT+: track 198.6 -> 209.2 mm, vias 8 -> 7
- net HPHONE: track 5.37 -> 0.00 mm
- net VOUT1: track 41.3 -> 37.6 mm
- net VIN1: track 31.3 -> 33.3 mm
- net DC_VOL: track 69.5 -> 71.5 mm

Commit message: Fri  9 Mar 2018 22:54:46 EST - initial commit for sharing
Parts:
- moved C10 3.00 mm to (22.0, 5.00)
- moved C1 1.57 mm to (22.0, 7.95)
Routing:
- net BYP: track 4.41 -> 7.41 mm
- net VIN1: track 33.3 -> 31.3 mm
- net VOUT2: track 38.3 -> 37.3 mm
- net GND: vias 8 -> 9
Other:
- board text added: "100uF 220nF 1uF 1uF 100K 150Ohm LM4875"
- board text added: "C1 C2 C10 C12 R3 R4 U1"
- board text removed: "100uF 220nF 1uF 1uF 1KOhm 150Ohm 1KOhm LM4875"
- board text removed: "C1 C2 C10 C12 R3 R4 R5 U1"
- board text removed: "R5"
