File: eagle/gameboy-pocket.sch (EAGLE design)
At the start: 33 parts, among them J1 AUDIO_JACK_3.5MM_PTH, U1 LM4875

Commit message: Tue Jan 30 17:53:42 EST 2018
Connections:
- net DC_VOL: now also R10.E; no longer R10.S
- net SWITCH_OUT+: now also R10.S; no longer R10.E
Changed lines of the file:
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@@
 <?xml version="1.0" encoding="utf-8"?>
 <!DOCTYPE eagle SYSTEM "eagle.dtd">
-<eagle version="8.5.0">
+<eagle version="8.4.1">
 <drawing>
 <settings>
@@
 </segment>
 <segment>
-<pinref part="R10" gate="R$1" pin="E"/>
-<wire x1="193.04" y1="15.24" x2="195.58" y2="15.24" width="0.1524" layer="91"/>
-<label x="195.58" y="15.24" size="1.016" layer="95"/>
-</segment>
-<segment>
 <pinref part="C12" gate="G$1" pin="1"/>
 <pinref part="C11" gate="G$1" pin="1"/>
@@
 <label x="284.48" y="40.64" size="1.016" layer="95"/>
 </segment>
+<segment>
+<pinref part="R10" gate="R$1" pin="S"/>
+<wire x1="187.96" y1="10.16" x2="195.58" y2="10.16" width="0.1524" layer="91"/>
+<label x="195.58" y="10.16" size="1.016" layer="95"/>
+</segment>
 </net>
 <net name="BATT+" class="0">
@@
 </segment>
 <segment>
-<pinref part="R10" gate="R$1" pin="S"/>
-<wire x1="187.96" y1="10.16" x2="195.58" y2="10.16" width="0.1524" layer="91"/>
-<label x="195.58" y="10.16" size="1.016" layer="95"/>
-</segment>
-</net>
+<pinref part="R10" gate="R$1" pin="E"/>
+<wire x1="193.04" y1="15.24" x2="195.58" y2="15.24" width="0.1524" layer="91"/>
+<label x="195.58" y="15.24" size="1.016" layer="95"/>
+</segment>
+</net>

Commit message: Wed 21 Feb 2018 12:43:42 EST
Parts:
- removed C11: 100nF, adafruit:C-USC0805
- removed C3: 220nF, adafruit:C-USC0805
- removed C4: 330nF, adafruit:C-USC0805
- removed J1: AUDIO_JACK_3.5MM_PTH, SparkFun-Connectors:AUDIO_JACK_3.5MM_PTH
- added C1: 100uF, adafruit:C-USC0805
- added R4: 150Ohm, adafruit:R-US_R0805
- added X1: STEREOJACK, adafruit:STEREOJACK
- C10: value 100nF -> 1uF
- C12: value 10uF -> 1uF
- C2: value 10uF -> 220nF; device SparkFun-Capacitors:10UF-POLAR-EIA3216-16V-10%(TANT) -> adafruit:C-USC0805
- R3, R5: value 270Ohm -> 1KOhm
Connections:
- removed net CAP_LINE: C11.2, C12.2, U1.VDD
- removed net CAP_LINE_JACK: C2.-, J1.RSH, J1.TSH
- removed net N$2: C3.2, C4.2, R3.2
- new net HPHONE: R5.1, U1.HPHONE
- new net VIN1: C1.2, R4.2, X1.2, X1.5
- net GND: now also C12.2, R4.1, X1.1; no longer C4.1, J1.SLEEVE
- net HEADPHONES: now also R3.1, R5.2, X1.3, X1.4; no longer J1.RING, J1.TIP, R5.1, U1.HPHONE
- net PWM: now also C2.2; no longer R3.1
- net SWITCH_OUT+: now also R3.2, U1.VDD; no longer C11.1, R5.2
- net VIN: now also C2.1; no longer C3.1
- net VOUT1: now also C1.1; no longer C2.+
Other:
- moved on the sheet: C10, C12, J2, R10, R3, R5
