File: eagle/Layout/GabozePocaioLayout.brd (EAGLE design)
At the start: 71.2 x 115.5 mm, 18 parts, among them J1 AUDIO_JACK_3.5MM_KIT, J2 Speaker

Commit message: Wed 27 Jun 2018 09:32:48 EDT
Parts:
- BTN_L1, BTN_R1, BTN_X, BTN_Y: value GAMEBOY-ZERO-BUTTON -> GAMEBOY-ZERO-BUTTON-DRILL; device GameboyZeroButtonLibrary:GAMEBOY-ZERO-BUTTON -> GameboyZeroButtonLibrary:GAMEBOY-ZERO-BUTTON-DRILL
- LED1: device adafruit:CHIPLED_0805 -> adafruit:LED3MM
- moved LED1 2.30 mm to (3.75, 99.5)
- moved R2 2.02 mm to (3.75, 103.0), turned to 0 degrees
Other:
- outline, holes or cut-outs redrawn
- board text added: "32teeth"

Commit message: Fri 29 Jun 2018 10:04:19 EDT
Parts:
- BTN_SELECT, BTN_START: value GAMEBOY-ZERO-BUTTON -> GAMEBOY-ZERO-BUTTON-STARTSELECT; device GameboyZeroButtonLibrary:GAMEBOY-ZERO-BUTTON -> GameboyZeroButtonLibrary:GAMEBOY-ZERO-BUTTON-STARTSELECT
Other:
- board text added: "a"
- board text added: "b"
