File: eagle/Layout/GabozePocaioLayout.brd (EAGLE design)
At the start: 71.2 x 115.5 mm, 18 parts, among them J1 AUDIO_JACK_3.5MM_KIT, J2 Speaker

Commit message: Mon  9 Jul 2018 07:06:11 EDT - updated layour eagle files
Parts:
- turned BTN_DOWN to 0 degrees
- turned BTN_UP to 180 degrees
Changed lines of the file:
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@@
 <?xml version="1.0" encoding="utf-8"?>
 <!DOCTYPE eagle SYSTEM "eagle.dtd">
-<eagle version="9.0.0">
+<eagle version="9.0.1">
 <drawing>
 <settings>
@@
 <element name="R2" library="adafruit" package="R0805" value="1.5K Ohms" x="3.75" y="103"/>
 <element name="LED1" library="adafruit" package="LED3MM" value="Red" x="3.75" y="99.5" rot="R180"/>
-<element name="BTN_UP" library="GameboyZeroButtonLibrary" package="GAMEBOY-ZERO-BUTTON" value="GAMEBOY-ZERO-BUTTON" x="12.2" y="44.9" smashed="yes" rot="R90">
-<attribute name="NAME" x="9.025" y="44.9" size="0.6096" layer="25" font="vector" ratio="20" rot="R90" align="bottom-center"/>
+<element name="BTN_UP" library="GameboyZeroButtonLibrary" package="GAMEBOY-ZERO-BUTTON" value="GAMEBOY-ZERO-BUTTON" x="12.2" y="44.9" smashed="yes" rot="R180">
+<attribute name="NAME" x="12.2" y="41.725" size="0.6096" layer="25" font="vector" ratio="20" rot="R180" align="bottom-center"/>
 </element>
-<element name="BTN_DOWN" library="GameboyZeroButtonLibrary" package="GAMEBOY-ZERO-BUTTON" value="GAMEBOY-ZERO-BUTTON" x="12.2" y="28.9" smashed="yes" rot="R270">
-<attribute name="NAME" x="15.375" y="28.9" size="0.6096" layer="25" font="vector" ratio="20" rot="R270" align="bottom-center"/>
+<element name="BTN_DOWN" library="GameboyZeroButtonLibrary" package="GAMEBOY-ZERO-BUTTON" value="GAMEBOY-ZERO-BUTTON" x="12.2" y="28.9" smashed="yes">
+<attribute name="NAME" x="12.2" y="32.075" size="0.6096" layer="25" font="vector" ratio="20" align="bottom-center"/>
 </element>
 <element name="BTN_LEFT" library="GameboyZeroButtonLibrary" package="GAMEBOY-ZERO-BUTTON" value="GAMEBOY-ZERO-BUTTON" x="4.2" y="36.9" smashed="yes" rot="R90">
