File: eagle/Layout/GabozePocaioLayout.brd (EAGLE design)
At the start: 71.2 x 115.5 mm, 18 parts, among them J1 AUDIO_JACK_3.5MM_KIT, J2 Speaker

Commit message: Fri 13 Jul 2018 07:20:31 EDT - updated layout eagle files with new buttons
Parts:
- removed LED1: Red, adafruit:LED3MM
- removed R2: 1.5K Ohms, adafruit:R0805
- added J4: ZX62-B-5PA, Seeed-Connector:MICRO-USB5+6P-SMD-0.65-AB
- J2: value Speaker -> SPKR
- turned BTN_DOWN to 90 degrees
- turned BTN_LEFT to 0 degrees
- turned BTN_RIGHT to 0 degrees
- turned BTN_UP to 90 degrees
Other:
- outline, holes or cut-outs redrawn
- board text removed: "a"
- board text removed: "b"
