File: eagle/Layout/GabozePocaioLayout.sch (EAGLE design)
At the start: 18 parts, among them J1 AUDIO_JACK_3.5MM_KIT, J2 Speaker

Commit message: Fri 13 Jul 2018 07:20:31 EDT - updated layout eagle files with new buttons
Parts:
- removed LED1: Red, adafruit:LED3MM
- removed R2: 1.5K Ohms, adafruit:R-US_R0805
- added J4: ZX62-B-5PA, Seeed-Connector:MICRO-USB-SMD(ZX62-B-5PA)
- J2: value Speaker -> SPKR
Other:
- note added: "CREDITS"
- moved on the sheet: U$1
Changed lines of the file:
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@@
 <part name="BTN_A" library="ConductiveButtons" deviceset="CONDUCTIVE_BUTTON" device="" value="CONDUCTIVE_BUTTON"/>
 <part name="BTN_R1" library="ConductiveButtons" deviceset="CONDUCTIVE_BUTTON_DRILL" device="" value="CONDUCTIVE_BUTTON_DRILL"/>
-<part name="R2" library="adafruit" deviceset="R-US_" device="R0805" value="1.5K Ohms"/>
-<part name="LED1" library="adafruit" deviceset="LED" device="3MM" value="Red"/>
 <part name="BTN_UP" library="ConductiveButtons" deviceset="CONDUCTIVE_BUTTON" device="" value="CONDUCTIVE_BUTTON"/>
 <part name="BTN_DOWN" library="ConductiveButtons" deviceset="CONDUCTIVE_BUTTON" device="" value="CONDUCTIVE_BUTTON"/>
@@
 <part name="U$1" library="SparkFun-Retired" library_urn="urn:adsk.eagle:library:533" deviceset="SWITCH_SPDT" device=""/>
 <part name="R10" library="GBA" deviceset="VOLUME" device="" value="27k"/>
-<part name="J2" library="SparkFun-Connectors" library_urn="urn:adsk.eagle:library:513" deviceset="CONN_02" device="" package3d_urn="urn:adsk.eagle:package:38039/1" value="Speaker"/>
+<part name="J2" library="SparkFun-Connectors" library_urn="urn:adsk.eagle:library:513" deviceset="CONN_02" device="" package3d_urn="urn:adsk.eagle:package:38039/1" value="SPKR"/>
+<part name="J4" library="Seeed-Connector" library_urn="urn:adsk.eagle:library:478" deviceset="MICRO-USB-SMD(ZX62-B-5PA)" device="" package3d_urn="urn:adsk.eagle:package:33147/1" value="ZX62-B-5PA"/>
 <part name="J1" library="SparkFun-Connectors" library_urn="urn:adsk.eagle:library:513" deviceset="AUDIO_JACK_3.5MM" device="_KIT" package3d_urn="urn:adsk.eagle:package:38014/1"/>
 </parts>
@@
 <wire x1="77.851" y1="143.51" x2="3.81" y2="143.51" width="0" layer="94"/>
 <text x="40.64" y="145.796" size="1.016" layer="94" font="vector" align="center">BATTERY</text>
-<wire x1="151.765" y1="3.81" x2="151.765" y2="22.86" width="0" layer="94"/>
-<wire x1="151.765" y1="22.86" x2="151.765" y2="27.94" width="0" layer="94"/>
-<wire x1="151.765" y1="27.94" x2="77.724" y2="27.94" width="0" layer="94"/>
-<wire x1="151.765" y1="22.86" x2="77.724" y2="22.86" width="0" layer="94"/>
-<text x="114.554" y="25.146" size="1.016" layer="94" font="vector" align="center">SWITCH</text>
-<wire x1="151.765" y1="27.94" x2="151.765" y2="46.99" width="0" layer="94"/>
+<wire x1="151.765" y1="3.81" x2="151.765" y2="46.99" width="0" layer="94"/>
+<text x="289.814" y="121.666" size="1.016" layer="94" font="vector" align="center">SWITCH</text>
 <wire x1="151.765" y1="46.99" x2="151.765" y2="52.07" width="0" layer="94"/>
-<wire x1="151.765" y1="52.07" x2="77.724" y2="52.07" width="0" layer="94"/>
-<text x="114.554" y="49.276" size="1.016" layer="94" font="vector" align="center">LED</text>
-<wire x1="151.765" y1="46.99" x2="77.724" y2="46.99" width="0" layer="94"/>
+<text x="289.814" y="145.796" size="1.016" layer="94" font="vector" align="center">LED</text>
 <wire x1="151.765" y1="52.07" x2="151.765" y2="124.46" width="0" layer="94"/>
 <wire x1="151.765" y1="76.2" x2="151.765" y2="143.51" width="0" layer="94"/>
@@
 <wire x1="250.571" y1="143.51" x2="151.765" y2="143.51" width="0" layer="94"/>
 <wire x1="250.571" y1="143.51" x2="250.571" y2="148.59" width="0" layer="94"/>
-<wire x1="324.231" y1="52.07" x2="151.765" y2="52.07" width="0" layer="94"/>
+<wire x1="324.231" y1="52.07" x2="250.571" y2="52.07" width="0" layer="94"/>
+<wire x1="250.571" y1="52.07" x2="151.765" y2="52.07" width="0" layer="94"/>
 <wire x1="324.231" y1="46.99" x2="151.765" y2="46.99" width="0" layer="94"/>
 <text x="244.094" y="49.276" size="1.016" layer="94" font="vector" align="center">AUDIO</text>
 <wire x1="324.231" y1="143.51" x2="250.571" y2="143.51" width="0" layer="94"/>
-<text x="289.56" y="145.796" size="1.016" layer="94" font="vector" align="center">RASPBERRY PI</text>
+<wire x1="324.485" y1="124.46" x2="250.571" y2="124.46" width="0" layer="94"/>
+<wire x1="324.485" y1="100.33" x2="250.825" y2="100.33" width="0" layer="94"/>
+<wire x1="250.571" y1="52.07" x2="250.571" y2="119.38" width="0" layer="94"/>
+<wire x1="250.571" y1="119.38" x2="250.571" y2="124.46" width="0" layer="94"/>
+<wire x1="250.571" y1="124.46" x2="250.571" y2="143.51" width="0" layer="94"/>
+<wire x1="324.485" y1="95.25" x2="250.825" y2="95.25" width="0" layer="94"/>
+<wire x1="324.485" y1="119.38" x2="250.571" y2="119.38" width="0" layer="94"/>
+<text x="289.814" y="97.536" size="1.016" layer="94" font="vector" align="center">CREDITS</text>
 </plain>
 <instances>
@@
 <attribute name="NAME" x="55.88" y="59.182" size="1.016" layer="95" font="vector" align="bottom-center"/>
 </instance>
-<instance part="R2" gate="G$1" x="124.46" y="38.1"/>
-<instance part="LED1" gate="G$1" x="111.76" y="38.1" rot="R270"/>
 <instance part="BTN_UP" gate="G$1" x="25.4" y="16.51" smashed="yes">
 <attribute name="NAME" x="25.4" y="18.034" size="1.016" layer="95" font="vector" align="bottom-center"/>
@@
 <attribute name="NAME" x="55.88" y="18.034" size="1.016" layer="95" font="vector" align="bottom-center"/>
 </instance>
-<instance part="U$1" gate="G$1" x="114.3" y="12.7"/>
+<instance part="U$1" gate="G$1" x="289.56" y="109.22"/>
 <instance part="R10" gate="R$1" x="185.42" y="25.4" rot="R270"/>
 <instance part="J2" gate="G$1" x="317.5" y="40.64" rot="R180"/>
+<instance part="J4" gate="G$1" x="17.526" y="109.728"/>
 <instance part="J1" gate="G$1" x="307.34" y="12.7" rot="R180"/>
 </instances>
